File: Hardware/Microphone_Breakout_Board.kicad_pcb (KiCad board)
At the start: 2 copper layers, 20 x 20 mm, 5 parts, among them J1 Conn_01x04

Commit message: Routed PCB.
Parts:
- C1, C2, C3: footprint Capacitor_SMD:C_0603_1608Metric_Pad1.08x0.95mm_HandSolder -> Capacitor_SMD:C_1206_3216Metric
- moved C1 2.44 mm to (186.1, 89.5), turned to 180 degrees
- moved C2 1.28 mm to (191.6, 98.4)
- moved C3 0.65 mm to (191.6, 95.9)
Routing:
- net VDD: track 0.00 -> 11.7 mm
- net Net-(C2-Pad2): track 0.00 -> 6.91 mm
- net Net-(C2-Pad1): track 0.00 -> 4.49 mm
- net Net-(C3-Pad1): track 0.00 -> 4.23 mm
- net Net-(C3-Pad2): track 0.00 -> 3.23 mm
- added copper zone on F.Cu, net GND
Other:
- board text added: "SPW0878LR5H-1 Ellen Microphone board"

Commit message: Added manufacturing data to schematic and PCB.
Changed lines of the file:
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@@
   )
   (setup
-    (last_trace_width 1)
+    (last_trace_width 0.25)
     (user_trace_width 0.36)
     (user_trace_width 1)
@@
     (pad_drill 0.762)
     (pad_to_mask_clearance 0)
-    (aux_axis_origin 0 0)
+    (aux_axis_origin 181 103)
+    (grid_origin 181 103)
     (visible_elements FFFFFF7F)
     (pcbplotparams
@@
       (outputformat 1)
       (mirror false)
-      (drillshape 1)
+      (drillshape 0)
       (scaleselection 1)
-      (outputdirectory ""))
+      (outputdirectory "Production_Files/"))
   )
   (net 0 "")
@@
       (effects (font (size 1 1) (thickness 0.15)))
     )
-    (fp_text user %R (at 0 0) (layer F.Fab)
-      (effects (font (size 0.8 0.8) (thickness 0.12)))
-    )
     (fp_line (start -1.6 0.8) (end -1.6 -0.8) (layer F.Fab) (width 0.1))
     (fp_line (start -1.6 -0.8) (end 1.6 -0.8) (layer F.Fab) (width 0.1))
@@
     (fp_line (start 2.3 -1.15) (end 2.3 1.15) (layer F.CrtYd) (width 0.05))
     (fp_line (start 2.3 1.15) (end -2.3 1.15) (layer F.CrtYd) (width 0.05))
-    (pad 2 smd roundrect (at 1.475 0 180) (size 1.15 1.8) (layers F.Cu F.Paste F.Mask) (roundrect_rratio 0.217391)
+    (fp_text user %R (at 0 0) (layer F.Fab)
+      (effects (font (size 0.8 0.8) (thickness 0.12)))
+    )
+    (pad 2 smd roundrect (at 1.475 0 180) (size 1.15 1.8) (layers F.Cu F.Paste F.Mask) (roundrect_rratio 0.2173904347826087)
       (net 5 "Net-(C3-Pad2)"))
-    (pad 1 smd roundrect (at -1.475 0 180) (size 1.15 1.8) (layers F.Cu F.Paste F.Mask) (roundrect_rratio 0.217391)
+    (pad 1 smd roundrect (at -1.475 0 180) (size 1.15 1.8) (layers F.Cu F.Paste F.Mask) (roundrect_rratio 0.2173904347826087)
       (net 6 "Net-(C3-Pad1)"))
     (model ${KISYS3DMOD}/Capacitor_SMD.3dshapes/C_1206_3216Metric.wrl
@@
       (effects (font (size 0.8 0.8) (thickness 0.12)))
     )
-    (pad 1 smd roundrect (at -1.475 0 180) (size 1.15 1.8) (layers F.Cu F.Paste F.Mask) (roundrect_rratio 0.217391)
+    (pad 1 smd roundrect (at -1.475 0 180) (size 1.15 1.8) (layers F.Cu F.Paste F.Mask) (roundrect_rratio 0.2173904347826087)
       (net 4 "Net-(C2-Pad1)"))
-    (pad 2 smd roundrect (at 1.475 0 180) (size 1.15 1.8) (layers F.Cu F.Paste F.Mask) (roundrect_rratio 0.217391)
+    (pad 2 smd roundrect (at 1.475 0 180) (size 1.15 1.8) (layers F.Cu F.Paste F.Mask) (roundrect_rratio 0.2173904347826087)
       (net 3 "Net-(C2-Pad2)"))
     (model ${KISYS3DMOD}/Capacitor_SMD.3dshapes/C_1206_3216Metric.wrl
@@
     (fp_text value 100n (at 0 1.85) (layer F.Fab) hide
       (effects (font (size 1 1) (thickness 0.15)))
-    )
-    (fp_text user %R (at 0 0) (layer F.Fab)
-      (effects (font (size 0.8 0.8) (thickness 0.12)))
     )
     (fp_line (start -1.6 0.8) (end -1.6 -0.8) (layer F.Fab) (width 0.1))
@@
     (fp_line (start 2.3 -1.15) (end 2.3 1.15) (layer F.CrtYd) (width 0.05))
     (fp_line (start 2.3 1.15) (end -2.3 1.15) (layer F.CrtYd) (width 0.05))
-    (pad 2 smd roundrect (at 1.475 0 180) (size 1.15 1.8) (layers F.Cu F.Paste F.Mask) (roundrect_rratio 0.217391)
+    (fp_text user %R (at 0 0) (layer F.Fab)
+      (effects (font (size 0.8 0.8) (thickness 0.12)))
+    )
+    (pad 2 smd roundrect (at 1.475 0 180) (size 1.15 1.8) (layers F.Cu F.Paste F.Mask) (roundrect_rratio 0.2173904347826087)
       (net 1 GND))
-    (pad 1 smd roundrect (at -1.475 0 180) (size 1.15 1.8) (layers F.Cu F.Paste F.Mask) (roundrect_rratio 0.217391)
+    (pad 1 smd roundrect (at -1.475 0 180) (size 1.15 1.8) (layers F.Cu F.Paste F.Mask) (roundrect_rratio 0.2173904347826087)
       (net 2 VDD))
     (model ${KISYS3DMOD}/Capacitor_SMD.3dshapes/C_1206_3216Metric.wrl
@@
     )
     (fp_text value Conn_01x04 (at 4.385 -9.89) (layer B.Fab) hide
-      (effects (font (size 1 1) (thickness 0.15)) (justify mirror))
-    )
-    (fp_text user %R (at 2.77 -3.81 -90) (layer B.Fab)
       (effects (font (size 1 1) (thickness 0.15)) (justify mirror))
     )
@@
     (fp_line (start 10.55 -9.4) (end 10.55 1.8) (layer B.CrtYd) (width 0.05))
     (fp_line (start 10.55 1.8) (end -1.8 1.8) (layer B.CrtYd) (width 0.05))
+    (fp_text user %R (at 2.77 -3.81 -90) (layer B.Fab)
+      (effects (font (size 1 1) (thickness 0.15)) (justify mirror))
+    )
     (pad 4 thru_hole oval (at 0 -7.62) (size 1.7 1.7) (drill 1) (layers *.Cu *.Mask)
       (net 2 VDD))
